File: T24-BBB/T24-BBB.kicad_pcb (KiCad board)
At the start: 2 copper layers, 195.3 x 127.1 mm, 206 parts, among them J1 Port 1, J10 Port 10, J11 Port 11, J12 Port 12, J13 Port 13, J14 Port 14, J15 Port 15, J16 Port 16, J17 Port 17, J18 Port 18, J19 Port 19, J2 Port 2, J20 Port 20, J21 Port 21, J22 Port 22, J23 Port 23, J24 Port 24, J25 9-16 In, J26 1-8 In, J27 17-24 In, J28 5V In, J29 OLED, J3 Port 3, J30 5V Select, J31 VIN2_V, J32 VIN3_V, J33 VIN1_V, J34 25-28, J35 29-32, J36 33-36, J37 37-40, J38 41-44, J4 Port 4, J40 DMX2, J41 DMX1, J44 GPIO, J5 Port 5, J6 Port 6, J7 Port 7, J8 Port 8, J9 Port 9, SW2 Enter BTN, SW3 Down BTN, U1 74HC245D, U10 Buck, U11 BEAGLEBONEBLACK, U17 74HC245D, U2 AT24C256C, U3 AM26LS31CDR, U4 AM26LS31CDR, U5 AM26LS31CDR, U6 AM26LS31CDR, U7 AM26LS31CDR, U8 UA9638CD, U9 74HC245D

Commit message: SD Bus & Plugs
Fix GPIO and buttons sharing SD pins. Fix spacing on plugs as too tight.
Parts:
- moved C8 17.7 mm to (102.3, 127.8)
- moved U8 17.7 mm to (97.5, 124.9)
- moved J8 5.49 mm to (86.1, 121.4)
- moved J6 5.06 mm to (86.1, 105.5)
- moved J4 4.64 mm to (86.1, 89.5)
- moved J10 4.36 mm to (120.2, 124.8)
- moved J12 4.36 mm to (135.6, 124.8)
- moved J16 4.36 mm to (166.5, 124.8)
- moved J18 4.36 mm to (195.7, 124.9)
- moved J20 4.36 mm to (211.1, 124.9)
- moved J22 4.36 mm to (226.6, 124.9)
- moved J24 4.36 mm to (242.0, 124.9)
- moved J14 4.36 mm to (151.0, 124.8)
- moved J2 4.25 mm to (86.1, 73.6)
- moved R27 1.95 mm to (175.1, 132.5)
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Connections:
- U11 pad P8_11: (no net) -> GPIO1
- U11 pad P8_13: DATA25 -> BTN2
- U11 pad P8_15: (no net) -> DATA25
- U11 pad P8_16: (no net) -> BTN1
- U11 pad P8_3: GPIO1 -> (no net)
- U11 pad P8_4: GPIO2 -> (no net)
- U11 pad P8_5: BTN1 -> (no net)
- U11 pad P8_6: BTN2 -> (no net)
- U11 pad P8_7: DATA23 -> GPIO2
- U11 pad P8_8: (no net) -> DATA23
Routing:
- net Net-(J41-Pad3): track 24.5 -> 45.8 mm
- net Net-(J41-Pad2): track 17.9 -> 37.3 mm
- net Net-(J40-Pad2): track 29.0 -> 48.3 mm
- net Net-(J40-Pad1): track 25.9 -> 44.9 mm
- net SER1: track 161.5 -> 143.1 mm
- net SER2: track 161.5 -> 143.2 mm
- net +5V: track 599.1 -> 581.6 mm
- net Net-(J2-Pad2): track 22.7 -> 32.3 mm
- net BTN1: track 23.0 -> 16.0 mm
- net Net-(D17-Pad2): track 39.9 -> 33.0 mm
- net GPIO1: track 8.60 -> 14.8 mm
- net Net-(D29-Pad2): track 39.9 -> 33.9 mm
- net Net-(D28-Pad2): track 24.2 -> 18.8 mm
- net Net-(D26-Pad2): track 24.1 -> 19.0 mm
- net Net-(D30-Pad2): track 23.6 -> 18.6 mm
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
Commit message: Bump to 0.7b
Changed DMX connector. Tweaks.
Parts:
- added G***: LOGO, 3544again:beagle, F.Cu at (133.0, 71.3)
- added G***: LOGO, 3544again:logo1612, F.Cu at (187.3, 53.2)
- J1, J10, J11, J12, J13, J14, J15, J16, J17, J18, J19, J2, J20, J21, J22, J23, J24, J3, J4, J5, J6, J7, J8, J9: footprint 3544again:TimPheonix -> Connector_Phoenix_MC:PhoenixContact_MCV_1,5_3-G-3.5_1x03_P3.50mm_Vertical
- J41: footprint TerminalBlock_MetzConnect:TerminalBlock_MetzConnect_Type101_RT01604HBWC_1x04_P5.08mm_Horizontal -> Connector_Phoenix_MC:PhoenixContact_MCV_1,5_4-G-3.5_1x04_P3.50mm_Vertical
- R25, R26, R27, R28, R52, R53, R54, R55, R56, R57, R58, R59, R60, R61, R62, R63, R64, R65, R66, R67, R68, R69, R70, R71, R72, R73, R74, R75: value 2.2k -> 4.7k
- moved J41 1.31 mm to (62.4, 133.8)
Routing:
- net Net-(F29-Pad2): track 26.6 -> 13.8 mm
- net GND: track 14.8 -> 20.7 mm, vias 194 -> 195
- net V5_In: track 36.3 -> 35.8 mm
- net Net-(J41-Pad3): track 45.8 -> 45.3 mm
Other:
- board text added: "Board: T24_5_2 V0.7b Details: https://github.com/Kosh42/PCB-Designs/T24-BBB Powered by FPP"
- board text removed: "Board: T24_5_2 V0.7 Details: https://github.com/Kosh42/PCB-Designs/T24-BBB Powered by FPP"
