File: T24-BBB/T24-BBB.sch (KiCad schematic (older format))
At the start: 38 parts, among them J25 9-16 In, J26 1-8 In, J27 17-24 In, J28 5V In, J29 OLED, J30 5V Select, J31 VIN2_V, J32 VIN3_V, J33 VIN1_V, J44 GPIO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

Commit message: 0.7
Buck and reroute
Parts:
- removed U10: Buck, Connector_PinHeader_2.54mm:PinHeader_1x03_P2.54mm_Vertical, symbol Converter_DCDC:OKI-78SR-5_1.5-W36-C
- added F25, F26, F27: 30A Max, 3544again:3544-2, symbol Device:Fuse
- added U10: MP1584, DC-BRICK, symbol MP1584:MP1584
- F28: value 3A Max -> 2A Max
- J28: value 5V In -> Aux In
Connections:
- net labels added: Aux_In, V1, V2, V3
- net labels removed: V5_In
- no-connect marks 32 -> 28
Other:
- moved on the sheet: C2, J28, J30, R88, U2

Commit message: Updates. T24 to 7e
Changed lines of the file:
@@
 Sheet 1 6
 Title "T24"
-Date "2021-03-18"
-Rev "0.7d"
+Date "2021-04-13"
+Rev "0.7e"
 Comp "Lights On Windermere Avenue"
 Comment1 ""
@@
 GPIO2
 $Comp
-L Connector:Screw_Terminal_01x02 J26
-U 1 1 600E4B71
-P 1950 850
-F 0 "J26" H 2030 842 50  0000 L CNN
-F 1 "1-8 In" H 2030 751 50  0000 L CNN
-F 2 "TerminalBlock_MetzConnect:TerminalBlock_MetzConnect_Type701_RT11L02HGLU_1x02_P6.35mm_Horizontal" H 1950 850 50  0001 C CNN
-F 3 "~" H 1950 850 50  0001 C CNN
-	1    1950 850
-	1    0    0    1
-$EndComp
-$Comp
 L Connector:Screw_Terminal_01x02 J25
 U 1 1 600E5475
@@
 L Connector:Conn_01x02_Male J33
 U 1 1 602DD954
-P 950 1050
-F 0 "J33" V 900 1050 50  0000 R CNN
-F 1 "VIN1_V" V 800 1100 50  0000 R CNN
-F 2 "Connector_JST:JST_XH_B2B-XH-A_1x02_P2.50mm_Vertical" H 950 1050 50  0001 C CNN
-F 3 "~" H 950 1050 50  0001 C CNN
-	1    950  1050
-	0    -1   -1   0
+P 1050 1050
+F 0 "J33" V 1000 1050 50  0000 R CNN
+F 1 "VIN1_V" V 900 1100 50  0000 R CNN
+F 2 "Connector_JST:JST_XH_B2B-XH-A_1x02_P2.50mm_Vertical" H 1050 1050 50  0001 C CNN
+F 3 "~" H 1050 1050 50  0001 C CNN
+	1    1050 1050
+	0    1    -1   0
 $EndComp
 Wire Wire Line
@@
 Wire Wire Line
 	850  2700 1650 2700
-Connection ~ 1750 850
 Connection ~ 1650 1850
 Connection ~ 1650 2800
@@
 Text GLabel 3450 3150 3    50   Input ~ 0
 V3
+Connection ~ 1750 850
+$Comp
+L Connector:Screw_Terminal_01x02 J26
+U 1 1 600E4B71
+P 1950 850
+F 0 "J26" H 2030 842 50  0000 L CNN
+F 1 "1-8 In" H 2030 751 50  0000 L CNN
+F 2 "TerminalBlock_MetzConnect:TerminalBlock_MetzConnect_Type701_RT11L02HGLU_1x02_P6.35mm_Horizontal" H 1950 850 50  0001 C CNN
+F 3 "~" H 1950 850 50  0001 C CNN
+	1    1950 850
+	1    0    0    1
+$EndComp
 $EndSCHEMATC
