File: T24-BBB/DMX.sch (KiCad schematic (older format))
At the start: 7 parts, among them J40 DMX2, J41 DMX1, U8 UA9638CD

Commit message: Bump to 0.7b
Changed DMX connector. Tweaks.
Parts:
- J41: footprint TerminalBlock_MetzConnect:TerminalBlock_MetzConnect_Type101_RT01604HBWC_1x04_P5.08mm_Horizontal -> Connector_Phoenix_MC:PhoenixContact_MCV_1,5_4-G-3.5_1x04_P3.50mm_Vertical
Changed lines of the file:
@@
 Title "T24"
 Date "2021-03-14"
-Rev "0.7a"
+Rev "0.7b"
 Comp "Lights On Windermere Avenue"
 Comment1 ""
@@
 F 0 "J41" H 1818 1567 50  0000 C CNN
 F 1 "DMX1" H 1818 1476 50  0000 C CNN
-F 2 "TerminalBlock_MetzConnect:TerminalBlock_MetzConnect_Type101_RT01604HBWC_1x04_P5.08mm_Horizontal" H 1900 1250 50  0001 C CNN
+F 2 "Connector_Phoenix_MC:PhoenixContact_MCV_1,5_4-G-3.5_1x04_P3.50mm_Vertical" H 1900 1250 50  0001 C CNN
 F 3 "~" H 1900 1250 50  0001 C CNN
 	1    1900 1250
