File: T24-BBB/Ports 1 to 8.sch (KiCad schematic (older format))
At the start: 42 parts, among them J1 Port 1, J2 Port 2, J3 Port 3, J4 Port 4, J5 Port 5, J6 Port 6, J7 Port 7, J8 Port 8, U1 74HC245D

Commit message: Updates. T24 to 7e
Parts:
- J1, J2, J3, J4, J5, J6, J7, J8: footprint Connector_Phoenix_MC:PhoenixContact_MCV_1,5_3-G-3.5_1x03_P3.50mm_Vertical -> PhoenixContact_MCV_1,5_3-G-3.5_1x03_P3.50mm_Vertical_Tim
Changed lines of the file:
@@
 Sheet 2 6
 Title "T24"
-Date "2021-03-18"
-Rev "0.7d"
+Date "2021-04-13"
+Rev "0.7e"
 Comp "Lights On Windermere Avenue"
 Comment1 ""
@@
 F 0 "J1" V 3714 762 50  0000 R CNN
 F 1 "Port 1" V 3623 762 50  0000 R CNN
-F 2 "Connector_Phoenix_MC:PhoenixContact_MCV_1,5_3-G-3.5_1x03_P3.50mm_Vertical" H 3750 950 50  0001 C CNN
+F 2 "PhoenixContact_MCV_1,5_3-G-3.5_1x03_P3.50mm_Vertical_Tim" H 3750 950 50  0001 C CNN
 F 3 "~" H 3750 950 50  0001 C CNN
 	1    3750 950
@@
 F 0 "J2" V 4364 762 50  0000 R CNN
 F 1 "Port 2" V 4273 762 50  0000 R CNN
-F 2 "Connector_Phoenix_MC:PhoenixContact_MCV_1,5_3-G-3.5_1x03_P3.50mm_Vertical" H 4400 950 50  0001 C CNN
+F 2 "PhoenixContact_MCV_1,5_3-G-3.5_1x03_P3.50mm_Vertical_Tim" H 4400 950 50  0001 C CNN
 F 3 "~" H 4400 950 50  0001 C CNN
 	1    4400 950
@@
 F 0 "J3" V 5014 762 50  0000 R CNN
 F 1 "Port 3" V 4923 762 50  0000 R CNN
-F 2 "Connector_Phoenix_MC:PhoenixContact_MCV_1,5_3-G-3.5_1x03_P3.50mm_Vertical" H 5050 950 50  0001 C CNN
+F 2 "PhoenixContact_MCV_1,5_3-G-3.5_1x03_P3.50mm_Vertical_Tim" H 5050 950 50  0001 C CNN
 F 3 "~" H 5050 950 50  0001 C CNN
 	1    5050 950
@@
 F 0 "J4" V 5714 762 50  0000 R CNN
 F 1 "Port 4" V 5623 762 50  0000 R CNN
-F 2 "Connector_Phoenix_MC:PhoenixContact_MCV_1,5_3-G-3.5_1x03_P3.50mm_Vertical" H 5750 950 50  0001 C CNN
+F 2 "PhoenixContact_MCV_1,5_3-G-3.5_1x03_P3.50mm_Vertical_Tim" H 5750 950 50  0001 C CNN
 F 3 "~" H 5750 950 50  0001 C CNN
 	1    5750 950
@@
 F 0 "J5" V 6414 762 50  0000 R CNN
 F 1 "Port 5" V 6323 762 50  0000 R CNN
-F 2 "Connector_Phoenix_MC:PhoenixContact_MCV_1,5_3-G-3.5_1x03_P3.50mm_Vertical" H 6450 950 50  0001 C CNN
+F 2 "PhoenixContact_MCV_1,5_3-G-3.5_1x03_P3.50mm_Vertical_Tim" H 6450 950 50  0001 C CNN
 F 3 "~" H 6450 950 50  0001 C CNN
 	1    6450 950
@@
 F 0 "J6" V 7114 762 50  0000 R CNN
 F 1 "Port 6" V 7023 762 50  0000 R CNN
-F 2 "Connector_Phoenix_MC:PhoenixContact_MCV_1,5_3-G-3.5_1x03_P3.50mm_Vertical" H 7150 950 50  0001 C CNN
+F 2 "PhoenixContact_MCV_1,5_3-G-3.5_1x03_P3.50mm_Vertical_Tim" H 7150 950 50  0001 C CNN
 F 3 "~" H 7150 950 50  0001 C CNN
 	1    7150 950
@@
 F 0 "J7" V 7864 762 50  0000 R CNN
 F 1 "Port 7" V 7773 762 50  0000 R CNN
-F 2 "Connector_Phoenix_MC:PhoenixContact_MCV_1,5_3-G-3.5_1x03_P3.50mm_Vertical" H 7900 950 50  0001 C CNN
+F 2 "PhoenixContact_MCV_1,5_3-G-3.5_1x03_P3.50mm_Vertical_Tim" H 7900 950 50  0001 C CNN
 F 3 "~" H 7900 950 50  0001 C CNN
 	1    7900 950
@@
 F 0 "J8" V 8564 762 50  0000 R CNN
 F 1 "Port 8" V 8473 762 50  0000 R CNN
-F 2 "Connector_Phoenix_MC:PhoenixContact_MCV_1,5_3-G-3.5_1x03_P3.50mm_Vertical" H 8600 950 50  0001 C CNN
+F 2 "PhoenixContact_MCV_1,5_3-G-3.5_1x03_P3.50mm_Vertical_Tim" H 8600 950 50  0001 C CNN
 F 3 "~" H 8600 950 50  0001 C CNN
 	1    8600 950
