File: AB Connectons/Kosh's HartK/Kosh's HartK.sch (KiCad schematic (older format))
At the start: 8 parts, among them J1 HE_Heater, J2 HE Thrmistor, J3 Fans, J4 X_Carr, J7 Stepper, J8 MCU

Commit message: KoshABTool
Connections:
- net +24V: now also J8.10 (Pin_10); no longer J8.11 (Pin_11)
- net GNDA: now also J8.11 (Pin_11); no longer J8.1 (Pin_1)
- net HE_Fan_GND: now also J8.1 (Pin_1); no longer J8.2 (Pin_2)
- net Heat_GND: now also J8.9 (Pin_9); no longer J8.10 (Pin_10)
- net PC_Fan_GND: now also J8.8 (Pin_8); no longer J8.9 (Pin_9)
- net TH1: now also J8.12 (Pin_12); no longer J8.8 (Pin_8)
- net X_Stop: now also J8.2 (Pin_2); no longer J8.12 (Pin_12)
Changed lines of the file:
@@
 L power:+24V #PWR0104
 U 1 1 608635C3
-P 2750 2200
-F 0 "#PWR0104" H 2750 2050 50  0001 C CNN
-F 1 "+24V" V 2765 2328 50  0000 L CNN
-F 2 "" H 2750 2200 50  0001 C CNN
-F 3 "" H 2750 2200 50  0001 C CNN
-	1    2750 2200
-	0    -1   -1   0
+P 3250 2100
+F 0 "#PWR0104" H 3250 1950 50  0001 C CNN
+F 1 "+24V" V 3265 2228 50  0000 L CNN
+F 2 "" H 3250 2100 50  0001 C CNN
+F 3 "" H 3250 2100 50  0001 C CNN
+	1    3250 2100
+	0    1    1    0
 $EndComp
 $Comp
@@
 	0    -1   -1   0
 $EndComp
-Text GLabel 3250 2000 2    50   Input ~ 0
+Text GLabel 3250 2200 2    50   Input ~ 0
 TH1
-Text GLabel 3250 2100 2    50   Input ~ 0
+Text GLabel 2750 2100 0    50   Input ~ 0
 Heat_GND
 $Comp
@@
 Text GLabel 3250 2300 2    50   Input ~ 0
 ChT
+Text GLabel 2750 1700 0    50   Input ~ 0
+HE_Fan_GND
 Text GLabel 3250 1700 2    50   Input ~ 0
-HE_Fan_GND
-Text GLabel 3250 2200 2    50   Input ~ 0
 X_Stop
 $Comp
 L power:GNDA #PWR0112
 U 1 1 6086A991
-P 2750 1700
-F 0 "#PWR0112" H 2750 1450 50  0001 C CNN
-F 1 "GNDA" V 2755 1572 50  0000 R CNN
-F 2 "" H 2750 1700 50  0001 C CNN
-F 3 "" H 2750 1700 50  0001 C CNN
-	1    2750 1700
+P 2750 2200
+F 0 "#PWR0112" H 2750 1950 50  0001 C CNN
+F 1 "GNDA" V 2755 2072 50  0000 R CNN
+F 2 "" H 2750 2200 50  0001 C CNN
+F 3 "" H 2750 2200 50  0001 C CNN
+	1    2750 2200
 	0    1    1    0
 $EndComp
 Text GLabel 2750 2300 0    50   Input ~ 0
 ABL_MCU
-Text GLabel 2750 2100 0    50   Input ~ 0
+Text GLabel 3250 2000 2    50   Input ~ 0
 PC_Fan_GND
 Text GLabel 2750 2000 0    50   Input ~ 0
