File: Mirage/Mirage.kicad_pcb (KiCad board)
At the start: 2 copper layers, 195.3 x 127.1 mm, 209 parts, among them J1 Port 1, J10 Port 10, J11 Port 11, J12 Port 12, J13 Port 13, J14 Port 14, J15 Port 15, J16 Port 16, J17 Port 17, J18 Port 18, J19 Port 19, J2 Port 2, J20 Port 20, J21 Port 21, J22 Port 22, J23 Port 23, J24 Port 24, J25 9-16 In, J26 1-8 In, J27 17-24 In, J28 Aux In, J29 OLED, J3 Port 3, J30 5V Select, J31 VIN2_V, J32 VIN3_V, J33 VIN1_V, J34 25-28, J35 29-32, J36 33-36, J37 37-40, J38 41-44, J4 Port 4, J40 DMX2, J41 DMX1, J44 GPIO, J5 Port 5, J6 Port 6, J7 Port 7, J8 Port 8, J9 Port 9, SW2 Enter BTN, SW3 Down BTN, U1 74HC245D, U10 MP1584, U11 BEAGLEBONEBLACK, U17 74HC245D, U2 AT24C256C, U3 AM26LS31CDR, U4 AM26LS31CDR, U5 AM26LS31CDR, U6 AM26LS31CDR, U7 AM26LS31CDR, U8 UA9638CD, U9 74HC245D

Commit message: KoshABTool
Parts:
- added G***: LOGO, 3544again:logo1612, F.Cu at (115.5, 93.0)
- added REF**: OSHW-Logo2_14.6x12mm_SilkScreen, Symbol:OSHW-Logo2_14.6x12mm_SilkScreen, F.Cu at (188.1, 53.9)
- J1: value Port 1 -> G D V
- J10: value Port 10 -> G D V
- J11: value Port 11 -> G D V
- J12: value Port 12 -> G D V
- J13: value Port 13 -> G D V
- J14: value Port 14 -> G D V
- J15: value Port 15 -> G D V
- J16: value Port 16 -> G D V
- J17: value Port 17 -> G D V
- J18: value Port 18 -> G D V
- J19: value Port 19 -> G D V
- J2: value Port 2 -> G D V
- J20: value Port 20 -> G D V
- J21: value Port 21 -> G D V
- J22: value Port 22 -> G D V
- J23: value Port 23 -> G D V
- J24: value Port 24 -> G D V
- J3: value Port 3 -> G D V
- J4: value Port 4 -> G D V
- J5: value Port 5 -> G D V
- J6: value Port 6 -> G D V
- J7: value Port 7 -> G D V
- J8: value Port 8 -> G D V
- J9: value Port 9 -> G D V
- moved R23 0.07 mm to (228.5, 101.7)
Other:
- board text added: "Board: Mirage V1.0 Details: https://github.com/Kosh42/PCB-Designs/Mirage Powered by FPP"
- board text removed: "Board: T24 V0.7e Details: https://github.com/Kosh42/PCB-Designs/T24-BBB Powered by FPP"

Commit message: Updates
Add a few clean ups and upload settings JSON.
Routing:
- net Aux_In: track 47.4 -> 50.0 mm
- net Buck: track 63.7 -> 66.3 mm
Other:
- outline, holes or cut-outs redrawn
- board text added: "Board: Mirage V1.0a Details: https://github.com/Kosh42/PCB-Designs/Mirage Powered by FPP"
- board text removed: "Board: Mirage V1.0 Details: https://github.com/Kosh42/PCB-Designs/Mirage Powered by FPP"
Changed lines of the file:
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@@
   (general
     (thickness 1.6002)
-    (drawings 62)
-    (tracks 1883)
+    (drawings 63)
+    (tracks 1885)
     (zones 0)
     (modules 211)
@@
   )
   (setup
-    (last_trace_width 0.127)
+    (last_trace_width 4)
     (user_trace_width 0.15)
     (user_trace_width 0.2)
@@
     (add_net VIN3)
   )
+  (module MP1584:DC-BRICK (layer Front)
+    (at 207.22 28.73 270)
+    (fp_text reference U10 (at 2.015855 0 270) (layer F.SilkS)
+      (effects (font (size 0.787402 0.787402) (thickness 0.015)))
+    )
+    (fp_text value MP1584 (at 3.196958 0 270) (layer F.Fab)
+      (effects (font (size 0.787402 0.787402) (thickness 0.015)))
+    )
+    (fp_line (start 0 0) (end 22 0) (layer F.SilkS) (width 0.127))
+    (fp_line (start 0 0) (end 0 -17) (layer F.SilkS) (width 0.127))
+    (fp_line (start 0 -17) (end 22 -17) (layer F.SilkS) (width 0.127))
+    (fp_line (start 22 -17) (end 22 0) (layer F.SilkS) (width 0.127))
+    (fp_line (start 7.62 -8.89) (end 13.97 -8.89) (layer F.SilkS) (width 0.5))
+    (fp_line (start 13.97 -8.89) (end 12.7 -10.16) (layer F.SilkS) (width 0.5))
+    (fp_line (start 13.97 -8.89) (end 12.7 -7.62) (layer F.SilkS) (width 0.5))
+    (fp_text user OUT- (at 13.97 -12.7 270) (layer F.SilkS)
+      (effects (font (size 1 1) (thickness 0.015)))
+    )
+    (fp_text user OUT+ (at 13.97 -3.81 270) (layer F.SilkS)
+      (effects (font (size 1 1) (thickness 0.015)))
+    )
+    (fp_text user IN- (at 2.234452 -12.7 270) (layer F.SilkS)
+      (effects (font (size 1 1) (thickness 0.015)))
+    )
+    (fp_text user IN+ (at 3.81 -3.81 270) (layer F.SilkS)
+      (effects (font (size 1 1) (thickness 0.015)))
+    )
+    (pad OUT2+ thru_hole rect (at 20.5 -3.95 270) (size 1.308 1.308) (drill 0.8) (layers *.Cu *.Mask)
+      (net 205 Buck))
+    (pad OUT1+ thru_hole rect (at 20.5 -1.4 270) (size 1.308 1.308) (drill 0.8) (layers *.Cu *.Mask)
+      (net 205 Buck))
+    (pad OUT1 thru_hole rect (at 20.5 -13.4 270) (size 1.308 1.308) (drill 0.8) (layers *.Cu *.Mask)
+      (net 1 GND))
+    (pad OUT2 thru_hole rect (at 20.5 -15.87 270) (size 1.308 1.308) (drill 0.8) (layers *.Cu *.Mask)
+      (net 1 GND))
+    (pad IN1 thru_hole rect (at 1.5 -13.4 270) (size 1.308 1.308) (drill 0.8) (layers *.Cu *.Mask)
+      (net 1 GND))
+    (pad IN2 thru_hole rect (at 1.5 -15.87 270) (size 1.308 1.308) (drill 0.8) (layers *.Cu *.Mask)
+      (net 1 GND))
+    (pad IN2+ thru_hole rect (at 1.5 -3.95 270) (size 1.308 1.308) (drill 0.8) (layers *.Cu *.Mask)
+      (net 206 Aux_In))
+    (pad IN1+ thru_hole rect (at 1.5 -1.4 270) (size 1.308 1.308) (drill 0.8) (layers *.Cu *.Mask)
+      (net 206 Aux_In))
+  )
   (module 3544again:logo1612 (layer Front)
     (at 115.5 92.98)
@@
     )
   )
-  (module MP1584:DC-BRICK (layer Front)
-    (at 207.22 28.73 270)
-    (fp_text reference U10 (at 0 0 90) (layer F.SilkS)
-      (effects (font (size 0.787402 0.787402) (thickness 0.015)))
-    )
-    (fp_text value MP1584 (at 0 0 90) (layer F.Fab)
-      (effects (font (size 0.787402 0.787402) (thickness 0.015)))
-    )
-    (fp_line (start 0 0) (end 22 0) (layer F.SilkS) (width 0.127))
-    (fp_line (start 0 0) (end 0 -17) (layer F.SilkS) (width 0.127))
-    (fp_line (start 0 -17) (end 22 -17) (layer F.SilkS) (width 0.127))
-    (fp_line (start 22 -17) (end 22 0) (layer F.SilkS) (width 0.127))
-    (fp_line (start 7.62 -8.89) (end 13.97 -8.89) (layer F.SilkS) (width 0.5))
-    (fp_line (start 13.97 -8.89) (end 12.7 -10.16) (layer F.SilkS) (width 0.5))
-    (fp_line (start 13.97 -8.89) (end 12.7 -7.62) (layer F.SilkS) (width 0.5))
-    (fp_text user OUT- (at 13.97 -12.7 90) (layer F.SilkS)
-      (effects (font (size 1 1) (thickness 0.015)))
-    )
-    (fp_text user OUT+ (at 13.97 -3.81 90) (layer F.SilkS)
-      (effects (font (size 1 1) (thickness 0.015)))
-    )
-    (fp_text user IN- (at 3.81 -12.7 90) (layer F.SilkS)
-      (effects (font (size 1 1) (thickness 0.015)))
-    )
-    (fp_text user IN+ (at 3.81 -3.81 90) (layer F.SilkS)
-      (effects (font (size 1 1) (thickness 0.015)))
-    )
-    (pad OUT2+ thru_hole rect (at 20.5 -2.8 270) (size 1.308 1.308) (drill 0.8) (layers *.Cu *.Mask)
-      (net 205 Buck))
-    (pad OUT1+ thru_hole rect (at 20.5 -1.4 270) (size 1.308 1.308) (drill 0.8) (layers *.Cu *.Mask)
-      (net 205 Buck))
-    (pad OUT1 thru_hole rect (at 20.5 -14.47 270) (size 1.308 1.308) (drill 0.8) (layers *.Cu *.Mask)
-      (net 1 GND))
-    (pad OUT2 thru_hole rect (at 20.5 -15.87 270) (size 1.308 1.308) (drill 0.8) (layers *.Cu *.Mask)
-      (net 1 GND))
-    (pad IN1 thru_hole rect (at 1.5 -14.47 270) (size 1.308 1.308) (drill 0.8) (layers *.Cu *.Mask)
-      (net 1 GND))
-    (pad IN2 thru_hole rect (at 1.5 -15.87 270) (size 1.308 1.308) (drill 0.8) (layers *.Cu *.Mask)
-      (net 1 GND))
-    (pad IN2+ thru_hole rect (at 1.5 -2.8 270) (size 1.308 1.308) (drill 0.8) (layers *.Cu *.Mask)
-      (net 206 Aux_In))
-    (pad IN1+ thru_hole rect (at 1.5 -1.4 270) (size 1.308 1.308) (drill 0.8) (layers *.Cu *.Mask)
-      (net 206 Aux_In))
-  )
   (module Connector_RJ:RJ45_OST_PJ012-8P8CX_Vertical (layer Front)
     (at 110.9725 43.06 180)
@@
     )
   )
+  (gr_line (start 224.25 51.51) (end 225.09 50.67) (layer Edge.Cuts) (width 0.0381))
   (gr_circle (center 136.95 90.91) (end 136.96 90.91) (layer F.SilkS) (width 1))
   (gr_text "Inspired by https://github.com/computergeek1507/PB_16/\n\n" (at 171.57 104.06) (layer B.SilkS)
     (effects (font (size 1.524 1.524) (thickness 0.3048)) (justify mirror))
   )
-  (gr_line (start 225.09 51.51) (end 225.09 27.83) (layer Edge.Cuts) (width 0.0381))
-  (gr_line (start 200.52 51.51) (end 225.09 51.51) (layer Edge.Cuts) (width 0.0381))
+  (gr_line (start 225.09 50.67) (end 225.09 27.83) (layer Edge.Cuts) (width 0.0381))
+  (gr_line (start 200.52 51.51) (end 224.25 51.51) (layer Edge.Cuts) (width 0.0381))
   (gr_text "<12V Input" (at 188.32 30.91) (layer F.SilkS)
     (effects (font (size 1 1) (thickness 0.15)))
@@
   (gr_circle (center 184.55 66.92) (end 184.56 66.92) (layer F.SilkS) (width 1))
   (gr_line (start 197.24 54.79) (end 200.52 51.51) (layer Edge.Cuts) (width 0.0381))
-  (gr_text + (at 59.56 35.79 180) (layer F.SilkS)
+  (gr_text + (at 66.58 35.694 180) (layer F.SilkS)
     (effects (font (size 0.75 0.75) (thickness 0.1875)))
   )
@@
     (effects (font (size 0.75 0.75) (thickness 0.1875)))
   )
-  (gr_text - (at 66.71 35.7 180) (layer F.SilkS)
+  (gr_text - (at 60.23 35.7 180) (layer F.SilkS)
     (effects (font (size 0.75 0.75) (thickness 0.1875)))
   )
@@
     (effects (font (size 1 1) (thickness 0.15)))
   )
-  (gr_text "Board: Mirage V1.0\nDetails: https://github.com/Kosh42/PCB-Designs/Mirage\nPowered by FPP" (at 174.76 100.95) (layer F.SilkS)
+  (gr_text "Board: Mirage V1.0a\nDetails: https://github.com/Kosh42/PCB-Designs/Mirage\nPowered by FPP" (at 174.76 100.95) (layer F.SilkS)
     (effects (font (size 1.524 1.524) (thickness 0.3048)))
   )
@@
   (segment (start 184.305962 30.93) (end 183.868961 30.492999) (width 4) (layer Front) (net 205))
   (segment (start 203.26 30.93) (end 184.305962 30.93) (width 4) (layer Front) (net 205))
+  (segment (start 208.62 49.23) (end 211.17 49.23) (width 4) (layer Front) (net 205))
   (segment (start 196.51 37.46) (end 196.51 34.46) (width 4) (layer Back) (net 206))
   (segment (start 200.74 30.23) (end 210.02 30.23) (width 4) (layer Back) (net 206))
@@
   (segment (start 195.497001 36.447001) (end 182.44 36.447001) (width 4) (layer Front) (net 206))
   (segment (start 196.51 37.46) (end 195.497001 36.447001) (width 4) (layer Front) (net 206))
+  (segment (start 208.62 30.23) (end 211.17 30.23) (width 4) (layer Back) (net 206))
   (segment (start 69.333999 49.3547) (end 67.479299 47.5) (width 4) (layer Back) (net 239))
   (segment (start 69.333999 55.99) (end 69.333999 49.3547) (width 4) (layer Back) (net 239))
