File: Mirage/Mirage.sch (KiCad schematic (older format))
At the start: 41 parts, among them J25 9-16 In, J26 1-8 In, J27 17-24 In, J28 Aux In, J29 OLED, J30 5V Select, J31 VIN2_V, J32 VIN3_V, J33 VIN1_V, J44 GPIO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

Commit message: KoshABTool
Connections:
- net GND: now also J26.1 (Pin_1), J33.1 (Pin_1); no longer J26.2 (Pin_2), J33.2 (Pin_2)
- net V1: now also J26.2 (Pin_2), J33.2 (Pin_2); no longer J26.1 (Pin_1), J33.1 (Pin_1)
Changed lines of the file:
@@
 encoding utf-8
 Sheet 1 6
-Title "T24"
-Date "2021-04-13"
-Rev "0.7e"
+Title "Mirage"
+Date "2021-05-01"
+Rev "1.0"
 Comp "Lights On Windermere Avenue"
 Comment1 ""
@@
 GPIO2
 $Comp
-L Connector:Screw_Terminal_01x02 J26
-U 1 1 600E4B71
-P 1950 750
-F 0 "J26" H 2030 742 50  0000 L CNN
-F 1 "1-8 In" H 2030 651 50  0000 L CNN
-F 2 "TerminalBlock_MetzConnect:TerminalBlock_MetzConnect_Type701_RT11L02HGLU_1x02_P6.35mm_Horizontal" H 1950 750 50  0001 C CNN
-F 3 "~" H 1950 750 50  0001 C CNN
-	1    1950 750
-	1    0    0    -1
-$EndComp
-$Comp
 L Connector:Screw_Terminal_01x02 J25
 U 1 1 600E5475
@@
 L Connector:Conn_01x02_Male J33
 U 1 1 602DD954
-P 950 1050
-F 0 "J33" V 900 1050 50  0000 R CNN
-F 1 "VIN1_V" V 800 1100 50  0000 R CNN
-F 2 "Connector_JST:JST_XH_B2B-XH-A_1x02_P2.50mm_Vertical" H 950 1050 50  0001 C CNN
-F 3 "~" H 950 1050 50  0001 C CNN
-	1    950  1050
-	0    -1   -1   0
+P 1050 1050
+F 0 "J33" V 1000 1050 50  0000 R CNN
+F 1 "VIN1_V" V 900 1100 50  0000 R CNN
+F 2 "Connector_JST:JST_XH_B2B-XH-A_1x02_P2.50mm_Vertical" H 1050 1050 50  0001 C CNN
+F 3 "~" H 1050 1050 50  0001 C CNN
+	1    1050 1050
+	0    1    -1   0
 $EndComp
 Wire Wire Line
@@
 V3
 Connection ~ 1750 850
+$Comp
+L Connector:Screw_Terminal_01x02 J26
+U 1 1 600E4B71
+P 1950 850
+F 0 "J26" H 2030 842 50  0000 L CNN
+F 1 "1-8 In" H 2030 751 50  0000 L CNN
+F 2 "TerminalBlock_MetzConnect:TerminalBlock_MetzConnect_Type701_RT11L02HGLU_1x02_P6.35mm_Horizontal" H 1950 850 50  0001 C CNN
+F 3 "~" H 1950 850 50  0001 C CNN
+	1    1950 850
+	1    0    0    1
+$EndComp
 $EndSCHEMATC

Commit message: Updates
Add a few clean ups and upload settings JSON.
Parts:
- U10: symbol MP1584:MP1584 -> Mirage-rescue:MP1584-MP1584
- U11: symbol BBB:BEAGLEBONEBLACK -> Mirage-rescue:BEAGLEBONEBLACK-BBB
Changed lines of the file:
@@
 	950  1850 950  1750
 $Comp
-L BBB:BEAGLEBONEBLACK U11
+L Mirage-rescue:BEAGLEBONEBLACK-BBB U11
 U 1 1 601985F4
 P 9550 3600
@@
 Aux_In
 $Comp
-L MP1584:MP1584 U10
+L Mirage-rescue:MP1584-MP1584 U10
 U 1 1 6057B19B
 P 5400 4250
