File: Mirage/Ports 1 to 8.sch (KiCad schematic (older format))
At the start: 42 parts, among them J1 Port 1, J2 Port 2, J3 Port 3, J4 Port 4, J5 Port 5, J6 Port 6, J7 Port 7, J8 Port 8, U1 74HC245D

Commit message: KoshABTool
Parts:
- J1: value Port 1 -> G D V
- J2: value Port 2 -> G D V
- J3: value Port 3 -> G D V
- J4: value Port 4 -> G D V
- J5: value Port 5 -> G D V
- J6: value Port 6 -> G D V
- J7: value Port 7 -> G D V
- J8: value Port 8 -> G D V
Changed lines of the file:
@@
 encoding utf-8
 Sheet 2 6
-Title "T24"
-Date "2021-04-13"
-Rev "0.7e"
+Title "Mirage"
+Date "2021-05-01"
+Rev "1.0"
 Comp "Lights On Windermere Avenue"
 Comment1 ""
@@
 P 3750 950
 F 0 "J1" V 3714 762 50  0000 R CNN
-F 1 "Port 1" V 3623 762 50  0000 R CNN
+F 1 "G  D  V" V 3623 762 50  0000 R CNN
 F 2 "PhoenixContact_MCV_1,5_3-G-3.5_1x03_P3.50mm_Vertical_Tim" H 3750 950 50  0001 C CNN
 F 3 "~" H 3750 950 50  0001 C CNN
@@
 P 4400 950
 F 0 "J2" V 4364 762 50  0000 R CNN
-F 1 "Port 2" V 4273 762 50  0000 R CNN
+F 1 "G  D  V" V 4273 762 50  0000 R CNN
 F 2 "PhoenixContact_MCV_1,5_3-G-3.5_1x03_P3.50mm_Vertical_Tim" H 4400 950 50  0001 C CNN
 F 3 "~" H 4400 950 50  0001 C CNN
@@
 P 5050 950
 F 0 "J3" V 5014 762 50  0000 R CNN
-F 1 "Port 3" V 4923 762 50  0000 R CNN
+F 1 "G  D  V" V 4923 762 50  0000 R CNN
 F 2 "PhoenixContact_MCV_1,5_3-G-3.5_1x03_P3.50mm_Vertical_Tim" H 5050 950 50  0001 C CNN
 F 3 "~" H 5050 950 50  0001 C CNN
@@
 P 5750 950
 F 0 "J4" V 5714 762 50  0000 R CNN
-F 1 "Port 4" V 5623 762 50  0000 R CNN
+F 1 "G  D  V" V 5623 762 50  0000 R CNN
 F 2 "PhoenixContact_MCV_1,5_3-G-3.5_1x03_P3.50mm_Vertical_Tim" H 5750 950 50  0001 C CNN
 F 3 "~" H 5750 950 50  0001 C CNN
@@
 P 6450 950
 F 0 "J5" V 6414 762 50  0000 R CNN
-F 1 "Port 5" V 6323 762 50  0000 R CNN
+F 1 "G  D  V" V 6323 762 50  0000 R CNN
 F 2 "PhoenixContact_MCV_1,5_3-G-3.5_1x03_P3.50mm_Vertical_Tim" H 6450 950 50  0001 C CNN
 F 3 "~" H 6450 950 50  0001 C CNN
@@
 P 7150 950
 F 0 "J6" V 7114 762 50  0000 R CNN
-F 1 "Port 6" V 7023 762 50  0000 R CNN
+F 1 "G  D  V" V 7023 762 50  0000 R CNN
 F 2 "PhoenixContact_MCV_1,5_3-G-3.5_1x03_P3.50mm_Vertical_Tim" H 7150 950 50  0001 C CNN
 F 3 "~" H 7150 950 50  0001 C CNN
@@
 P 7900 950
 F 0 "J7" V 7864 762 50  0000 R CNN
-F 1 "Port 7" V 7773 762 50  0000 R CNN
+F 1 "G  D  V" V 7773 762 50  0000 R CNN
 F 2 "PhoenixContact_MCV_1,5_3-G-3.5_1x03_P3.50mm_Vertical_Tim" H 7900 950 50  0001 C CNN
 F 3 "~" H 7900 950 50  0001 C CNN
@@
 P 8600 950
 F 0 "J8" V 8564 762 50  0000 R CNN
-F 1 "Port 8" V 8473 762 50  0000 R CNN
+F 1 "G  D  V" V 8473 762 50  0000 R CNN
 F 2 "PhoenixContact_MCV_1,5_3-G-3.5_1x03_P3.50mm_Vertical_Tim" H 8600 950 50  0001 C CNN
 F 3 "~" H 8600 950 50  0001 C CNN

Commit message: Updates
Add a few clean ups and upload settings JSON.
Parts:
- U1: symbol SN74HCT245PW:SN74HCT245PW -> Mirage-rescue:SN74HCT245PW-SN74HCT245PW
Changed lines of the file:
@@
 $EndComp
 $Comp
-L SN74HCT245PW:SN74HCT245PW U1
+L Mirage-rescue:SN74HCT245PW-SN74HCT245PW U1
 U 1 1 6018FF62
 P 2350 2650
