File: Mirage/Ports 17 to 24.sch (KiCad schematic (older format))
At the start: 42 parts, among them J17 Port 17, J18 Port 18, J19 Port 19, J20 Port 20, J21 Port 21, J22 Port 22, J23 Port 23, J24 Port 24, U17 74HC245D

Commit message: KoshABTool
Parts:
- J17: value Port 17 -> G D V
- J18: value Port 18 -> G D V
- J19: value Port 19 -> G D V
- J20: value Port 20 -> G D V
- J21: value Port 21 -> G D V
- J22: value Port 22 -> G D V
- J23: value Port 23 -> G D V
- J24: value Port 24 -> G D V
Changed lines of the file:
@@
 encoding utf-8
 Sheet 4 6
-Title "T24"
-Date "2021-04-13"
-Rev "0.7e"
+Title "Mirage"
+Date "2021-05-01"
+Rev "1.0"
 Comp "Lights On Windermere Avenue"
 Comment1 ""
@@
 AR Path="/600DC29A/602077E6" Ref="J17"  Part="1"
 F 0 "J17" V 3464 812 50  0000 R CNN
-F 1 "Port 17" V 3373 812 50  0000 R CNN
+F 1 "G  D  V" V 3373 812 50  0000 R CNN
 F 2 "PhoenixContact_MCV_1,5_3-G-3.5_1x03_P3.50mm_Vertical_Tim" H 3500 1000 50  0001 C CNN
 F 3 "~" H 3500 1000 50  0001 C CNN
@@
 AR Path="/600DC29A/602077F3" Ref="J18"  Part="1"
 F 0 "J18" V 4114 812 50  0000 R CNN
-F 1 "Port 18" V 4023 812 50  0000 R CNN
+F 1 "G  D  V" V 4023 812 50  0000 R CNN
 F 2 "PhoenixContact_MCV_1,5_3-G-3.5_1x03_P3.50mm_Vertical_Tim" H 4150 1000 50  0001 C CNN
 F 3 "~" H 4150 1000 50  0001 C CNN
@@
 AR Path="/600DC29A/60207808" Ref="J19"  Part="1"
 F 0 "J19" V 4764 812 50  0000 R CNN
-F 1 "Port 19" V 4673 812 50  0000 R CNN
+F 1 "G  D  V" V 4673 812 50  0000 R CNN
 F 2 "PhoenixContact_MCV_1,5_3-G-3.5_1x03_P3.50mm_Vertical_Tim" H 4800 1000 50  0001 C CNN
 F 3 "~" H 4800 1000 50  0001 C CNN
@@
 AR Path="/600DC29A/6020781B" Ref="J20"  Part="1"
 F 0 "J20" V 5464 812 50  0000 R CNN
-F 1 "Port 20" V 5373 812 50  0000 R CNN
+F 1 "G  D  V" V 5373 812 50  0000 R CNN
 F 2 "PhoenixContact_MCV_1,5_3-G-3.5_1x03_P3.50mm_Vertical_Tim" H 5500 1000 50  0001 C CNN
 F 3 "~" H 5500 1000 50  0001 C CNN
@@
 AR Path="/600DC29A/6020782E" Ref="J21"  Part="1"
 F 0 "J21" V 6164 812 50  0000 R CNN
-F 1 "Port 21" V 6073 812 50  0000 R CNN
+F 1 "G  D  V" V 6073 812 50  0000 R CNN
 F 2 "PhoenixContact_MCV_1,5_3-G-3.5_1x03_P3.50mm_Vertical_Tim" H 6200 1000 50  0001 C CNN
 F 3 "~" H 6200 1000 50  0001 C CNN
@@
 AR Path="/600DC29A/60207841" Ref="J22"  Part="1"
 F 0 "J22" V 6864 812 50  0000 R CNN
-F 1 "Port 22" V 6773 812 50  0000 R CNN
+F 1 "G  D  V" V 6773 812 50  0000 R CNN
 F 2 "PhoenixContact_MCV_1,5_3-G-3.5_1x03_P3.50mm_Vertical_Tim" H 6900 1000 50  0001 C CNN
 F 3 "~" H 6900 1000 50  0001 C CNN
@@
 AR Path="/600DC29A/60207854" Ref="J23"  Part="1"
 F 0 "J23" V 7614 812 50  0000 R CNN
-F 1 "Port 23" V 7523 812 50  0000 R CNN
+F 1 "G  D  V" V 7523 812 50  0000 R CNN
 F 2 "PhoenixContact_MCV_1,5_3-G-3.5_1x03_P3.50mm_Vertical_Tim" H 7650 1000 50  0001 C CNN
 F 3 "~" H 7650 1000 50  0001 C CNN
@@
 AR Path="/600DC29A/60207867" Ref="J24"  Part="1"
 F 0 "J24" V 8314 812 50  0000 R CNN
-F 1 "Port 24" V 8223 812 50  0000 R CNN
+F 1 "G  D  V" V 8223 812 50  0000 R CNN
 F 2 "PhoenixContact_MCV_1,5_3-G-3.5_1x03_P3.50mm_Vertical_Tim" H 8350 1000 50  0001 C CNN
 F 3 "~" H 8350 1000 50  0001 C CNN

Commit message: Updates
Add a few clean ups and upload settings JSON.
Parts:
- U17: symbol SN74HCT245PW:SN74HCT245PW -> Mirage-rescue:SN74HCT245PW-SN74HCT245PW
Changed lines of the file:
@@
 $EndComp
 $Comp
-L SN74HCT245PW:SN74HCT245PW U?
+L Mirage-rescue:SN74HCT245PW-SN74HCT245PW U?
 U 1 1 60207774
 P 2100 2700
