File: Mirage/Ports 9 to 16.sch (KiCad schematic (older format))
At the start: 42 parts, among them J10 Port 10, J11 Port 11, J12 Port 12, J13 Port 13, J14 Port 14, J15 Port 15, J16 Port 16, J9 Port 9, U9 74HC245D

Commit message: KoshABTool
Parts:
- J10: value Port 10 -> G D V
- J11: value Port 11 -> G D V
- J12: value Port 12 -> G D V
- J13: value Port 13 -> G D V
- J14: value Port 14 -> G D V
- J15: value Port 15 -> G D V
- J16: value Port 16 -> G D V
- J9: value Port 9 -> G D V
Changed lines of the file:
@@
 encoding utf-8
 Sheet 3 6
-Title "T24"
-Date "2021-04-13"
-Rev "0.7e"
+Title "Mirage"
+Date "2021-05-01"
+Rev "1.0"
 Comp "Lights On Windermere Avenue"
 Comment1 ""
@@
 AR Path="/602A383B/602C12A3" Ref="J9"  Part="1"
 F 0 "J9" V 4614 1862 50  0000 R CNN
-F 1 "Port 9" V 4523 1862 50  0000 R CNN
+F 1 "G  D  V" V 4523 1862 50  0000 R CNN
 F 2 "PhoenixContact_MCV_1,5_3-G-3.5_1x03_P3.50mm_Vertical_Tim" H 4650 2050 50  0001 C CNN
 F 3 "~" H 4650 2050 50  0001 C CNN
@@
 AR Path="/602A383B/602C12B0" Ref="J10"  Part="1"
 F 0 "J10" V 5264 1862 50  0000 R CNN
-F 1 "Port 10" V 5173 1862 50  0000 R CNN
+F 1 "G  D  V" V 5173 1862 50  0000 R CNN
 F 2 "PhoenixContact_MCV_1,5_3-G-3.5_1x03_P3.50mm_Vertical_Tim" H 5300 2050 50  0001 C CNN
 F 3 "~" H 5300 2050 50  0001 C CNN
@@
 AR Path="/602A383B/602C12C5" Ref="J11"  Part="1"
 F 0 "J11" V 5914 1862 50  0000 R CNN
-F 1 "Port 11" V 5823 1862 50  0000 R CNN
+F 1 "G  D  V" V 5823 1862 50  0000 R CNN
 F 2 "PhoenixContact_MCV_1,5_3-G-3.5_1x03_P3.50mm_Vertical_Tim" H 5950 2050 50  0001 C CNN
 F 3 "~" H 5950 2050 50  0001 C CNN
@@
 AR Path="/602A383B/602C12D8" Ref="J12"  Part="1"
 F 0 "J12" V 6614 1862 50  0000 R CNN
-F 1 "Port 12" V 6523 1862 50  0000 R CNN
+F 1 "G  D  V" V 6523 1862 50  0000 R CNN
 F 2 "PhoenixContact_MCV_1,5_3-G-3.5_1x03_P3.50mm_Vertical_Tim" H 6650 2050 50  0001 C CNN
 F 3 "~" H 6650 2050 50  0001 C CNN
@@
 AR Path="/602A383B/602C12EB" Ref="J13"  Part="1"
 F 0 "J13" V 7314 1862 50  0000 R CNN
-F 1 "Port 13" V 7223 1862 50  0000 R CNN
+F 1 "G  D  V" V 7223 1862 50  0000 R CNN
 F 2 "PhoenixContact_MCV_1,5_3-G-3.5_1x03_P3.50mm_Vertical_Tim" H 7350 2050 50  0001 C CNN
 F 3 "~" H 7350 2050 50  0001 C CNN
@@
 AR Path="/602A383B/602C12FE" Ref="J14"  Part="1"
 F 0 "J14" V 8014 1862 50  0000 R CNN
-F 1 "Port 14" V 7923 1862 50  0000 R CNN
+F 1 "G  D  V" V 7923 1862 50  0000 R CNN
 F 2 "PhoenixContact_MCV_1,5_3-G-3.5_1x03_P3.50mm_Vertical_Tim" H 8050 2050 50  0001 C CNN
 F 3 "~" H 8050 2050 50  0001 C CNN
@@
 AR Path="/602A383B/602C1311" Ref="J15"  Part="1"
 F 0 "J15" V 8764 1862 50  0000 R CNN
-F 1 "Port 15" V 8673 1862 50  0000 R CNN
+F 1 "G  D  V" V 8673 1862 50  0000 R CNN
 F 2 "PhoenixContact_MCV_1,5_3-G-3.5_1x03_P3.50mm_Vertical_Tim" H 8800 2050 50  0001 C CNN
 F 3 "~" H 8800 2050 50  0001 C CNN
@@
 AR Path="/602A383B/602C1324" Ref="J16"  Part="1"
 F 0 "J16" V 9464 1862 50  0000 R CNN
-F 1 "Port 16" V 9373 1862 50  0000 R CNN
+F 1 "G  D  V" V 9373 1862 50  0000 R CNN
 F 2 "PhoenixContact_MCV_1,5_3-G-3.5_1x03_P3.50mm_Vertical_Tim" H 9500 2050 50  0001 C CNN
 F 3 "~" H 9500 2050 50  0001 C CNN

Commit message: Updates
Add a few clean ups and upload settings JSON.
Parts:
- U9: symbol SN74HCT245PW:SN74HCT245PW -> Mirage-rescue:SN74HCT245PW-SN74HCT245PW
Changed lines of the file:
@@
 $EndComp
 $Comp
-L SN74HCT245PW:SN74HCT245PW U?
+L Mirage-rescue:SN74HCT245PW-SN74HCT245PW U?
 U 1 1 602C1231
 P 3250 3750
